File: Zigzag 5p ATtiny connector.brd (EAGLE design)
At the start: 3 parts, among them J1 5 pin 0.05" ZIGZAG connector, U2 ATtiny3217

Commit message: Add files via upload
Parts:
- R1: device Albert:0603-SMALL -> Albert:0603
Changed lines of the file:
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@@
 <elements>
 <element name="U2" library="Albert-Arduino" package="QFN-24" value="ATtiny3217" x="5.207" y="5.461" smashed="yes"/>
-<element name="R1" library="Albert" package="0603-SMALL" value="100k" x="3.81" y="8.636" smashed="yes" rot="R270">
+<element name="R1" library="Albert" package="0603" value="100k" x="3.81" y="8.636" smashed="yes" rot="R270">
 <attribute name="VALUE" x="3.7465" y="9.8425" size="0.8128" layer="27" ratio="10" rot="R180" align="center"/>
 </element>
@@
 <contactref element="J1" pad="3"/>
 <wire x1="4.457" y1="7.461" x2="8.7122" y2="5.08" width="0" layer="19" extent="1-1"/>
-<wire x1="4.51" y1="8.636" x2="4.457" y2="7.461" width="0" layer="19" extent="1-1"/>
+<wire x1="4.56" y1="8.636" x2="4.457" y2="7.461" width="0" layer="19" extent="1-1"/>
 </signal>
 <signal name="VCC">
@@
 <contactref element="U2" pad="4"/>
 <contactref element="J1" pad="2"/>
-<wire x1="3.207" y1="5.211" x2="3.11" y2="8.636" width="0" layer="19" extent="1-1"/>
+<wire x1="3.207" y1="5.211" x2="3.06" y2="8.636" width="0" layer="19" extent="1-1"/>
 <wire x1="9.0678" y1="3.81" x2="3.207" y2="5.211" width="0" layer="19" extent="1-1"/>
 </signal>
