File: Zigzag 5p ATtiny connector.sch (EAGLE design)
At the start: 3 parts, among them J1 5 pin 0.05" ZIGZAG connector, U2 ATtiny3217

Commit message: Add files via upload
Parts:
- R1: device Albert:SMD-R0603-SMALL -> Albert:SMD-R0603
Changed lines of the file:
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@@
 <part name="U2" library="Albert-Arduino" deviceset="ATTINY3217" device="-" value="ATtiny3217"/>
 <part name="V5" library="Albert" deviceset="ARROW" device="" value="x"/>
-<part name="R1" library="Albert" deviceset="SMD-R" device="0603-SMALL" value="100k"/>
+<part name="R1" library="Albert" deviceset="SMD-R" device="0603" value="100k"/>
 <part name="GND3" library="Albert" deviceset="GND" device=""/>
 <part name="GND5" library="Albert" deviceset="GND" device=""/>
